File: Buffers.kicad_sch (KiCad schematic)
At the start: 85 parts, among them J301 FX_R_1, J302 FX_R_2, J303 FX_R_3, J304 FX_R_4, J305 FX_R_5, J306 FX_R_6, J307 FX_R_7, J308 FX_R_8, J309 FX_S_1, J310 FX_S_2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

Commit message: Removed LED Shift registers and replaced them with PCA9685 PWM controllers, Also changed LEDs to RGB LEDs.
Parts:
- renumbered C319 to C301, C327 to C302, C335 to C303, C301 to C304, C309 to C305, C317 to C306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
