File: pedal_routing_5-8.kicad_sch (KiCad schematic)
At the start: 14 parts, among them U601 CD4051B, U602 CD4051B, U603 CD4051B, U604 CD4051B

Commit message: Removed un-needed inhibit from amp out. thereby simplifying the shift registers.
Connections:
- net U902_Q0 renamed U901_Q4
- net U902_Q1 renamed U901_Q5
- net U902_Q2 renamed U901_Q6
- net U902_Q3 renamed U901_Q7
Changed lines of the file:
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@@
 		)
 	)
-	(label "U902_Q3"
+	(label "U901_Q7"
 		(at 31.75 139.7 0)
 		(effects
@@
 		)
 	)
-	(label "U902_Q2"
+	(label "U901_Q6"
 		(at 185.42 50.8 0)
 		(effects
@@
 		)
 	)
-	(label "U902_Q0"
+	(label "U901_Q4"
 		(at 38.1 50.8 0)
 		(effects
@@
 		)
 	)
-	(label "U902_Q[0..3]"
+	(label "U901_Q[0..7]"
 		(at 16.51 78.74 0)
 		(effects
@@
 		)
 	)
-	(label "U902_Q1"
+	(label "U901_Q5"
 		(at 107.95 50.8 0)
 		(effects
@@
 		)
 	)
-	(hierarchical_label "U902_Q[0..3]"
+	(hierarchical_label "U901_Q[0..7]"
 		(shape output)
 		(at 16.51 69.85 0)

Commit message: Removed LED Shift registers and replaced them with PCA9685 PWM controllers, Also changed LEDs to RGB LEDs.
Parts:
- renumbered C604 to C601, C606 to C602, C608 to C603, C601 to C604, C607 to C605, C605 to C606, C603 to C607, C602 to C608, U603 to U602, U604 to U603, U602 to U604
Changed lines of the file:
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@@
 		(dnp no)
 		(fields_autoplaced yes)
-		(property "Reference" "U602"
+		(property "Reference" "U604"
 			(at 77.0733 119.38 0)
 			(effects
@@
 			(project "circuit"
 				(path "/420e3d7a-6c9a-4806-b4be-05d56aeb21de/badefe61-f2aa-4ce3-b43f-f44172d96524"
-					(reference "U602")
+					(reference "U604")
 					(unit 1)
 				)
@@
 		(dnp no)
 		(fields_autoplaced yes)
-		(property "Reference" "C608"
+		(property "Reference" "C603"
 			(at 236.2136 21.59 90)
 			(effects
@@
 			(project "circuit"
 				(path "/420e3d7a-6c9a-4806-b4be-05d56aeb21de/badefe61-f2aa-4ce3-b43f-f44172d96524"
-					(reference "C608")
+					(reference "C603")
 					(unit 1)
 				)
@@
 		(on_board yes)
 		(dnp no)
-		(property "Reference" "#PWR0606"
+		(property "Reference" "#PWR0602"
 			(at 179.07 34.29 0)
 			(effects
@@
 			(project "circuit"
 				(path "/420e3d7a-6c9a-4806-b4be-05d56aeb21de/badefe61-f2aa-4ce3-b43f-f44172d96524"
-					(reference "#PWR0606")
+					(reference "#PWR0602")
 					(unit 1)
 				)
@@
 		(dnp no)
 		(fields_autoplaced yes)
-		(property "Reference" "C607"
+		(property "Reference" "C605"
 			(at 210.8136 67.31 90)
 			(effects
@@
 			(project "circuit"
 				(path "/420e3d7a-6c9a-4806-b4be-05d56aeb21de/badefe61-f2aa-4ce3-b43f-f44172d96524"
-					(reference "C607")
+					(reference "C605")
 					(unit 1)
 				)
@@
 		(on_board yes)
 		(dnp no)
-		(property "Reference" "#PWR0601"
+		(property "Reference" "#PWR0604"
 			(at 54.61 91.44 0)
 			(effects
@@
 			(project "circuit"
 				(path "/420e3d7a-6c9a-4806-b4be-05d56aeb21de/badefe61-f2aa-4ce3-b43f-f44172d96524"
-					(reference "#PWR0601")
+					(reference "#PWR0604")
 					(unit 1)
 				)
@@
 		(on_board yes)
 		(dnp no)
-		(property "Reference" "#PWR0604"
+		(property "Reference" "#PWR0601"
 			(at 99.06 34.29 0)
 			(effects
@@
 			(project "circuit"
 				(path "/420e3d7a-6c9a-4806-b4be-05d56aeb21de/badefe61-f2aa-4ce3-b43f-f44172d96524"
-					(reference "#PWR0604")
+					(reference "#PWR0601")
 					(unit 1)
 				)
@@
 		(dnp no)
 		(fields_autoplaced yes)
-		(property "Reference" "C603"
+		(property "Reference" "C607"
 			(at 86.3536 110.49 90)
 			(effects
@@
 			(project "circuit"
 				(path "/420e3d7a-6c9a-4806-b4be-05d56aeb21de/badefe61-f2aa-4ce3-b43f-f44172d96524"
-					(reference "C603")
+					(reference "C607")
 					(unit 1)
 				)
@@
 		(dnp no)
 		(fields_autoplaced yes)
-		(property "Reference" "C602"
+		(property "Reference" "C608"
 			(at 60.9536 157.48 90)
 			(effects
@@
 			(project "circuit"
 				(path "/420e3d7a-6c9a-4806-b4be-05d56aeb21de/badefe61-f2aa-4ce3-b43f-f44172d96524"
-					(reference "C602")
+					(reference "C608")
 					(unit 1)
 				)
@@
 		(dnp no)
 		(fields_autoplaced yes)
-		(property "Reference" "C605"
+		(property "Reference" "C606"
 			(at 138.4236 68.58 90)
 			(effects
@@
 			(project "circuit"
 				(path "/420e3d7a-6c9a-4806-b4be-05d56aeb21de/badefe61-f2aa-4ce3-b43f-f44172d96524"
-					(reference "C605")
+					(reference "C606")
 					(unit 1)
 				)
@@
 		(dnp no)
 		(fields_autoplaced yes)
-		(property "Reference" "#FLG0602"
+		(property "Reference" "#FLG0601"
 			(at 27.94 33.655 0)
 			(effects
@@
 			(project ""
 				(path "/420e3d7a-6c9a-4806-b4be-05d56aeb21de/badefe61-f2aa-4ce3-b43f-f44172d96524"
-					(reference "#FLG0602")
+					(reference "#FLG0601")
 					(unit 1)
 				)
@@
 		(on_board yes)
 		(dnp no)
-		(property "Reference" "#PWR0608"
+		(property "Reference" "#PWR0603"
 			(at 246.38 34.29 0)
 			(effects
@@
 			(project "circuit"
 				(path "/420e3d7a-6c9a-4806-b4be-05d56aeb21de/badefe61-f2aa-4ce3-b43f-f44172d96524"
-					(reference "#PWR0608")
+					(reference "#PWR0603")
 					(unit 1)
 				)
@@
 		(dnp no)
 		(fields_autoplaced yes)
-		(property "Reference" "#FLG0601"
+		(property "Reference" "#FLG0602"
 			(at 74.93 74.295 0)
 			(effects
@@
 			(project ""
 				(path "/420e3d7a-6c9a-4806-b4be-05d56aeb21de/badefe61-f2aa-4ce3-b43f-f44172d96524"
-					(reference "#FLG0601")
+					(reference "#FLG0602")
 					(unit 1)
 				)
@@
 		(dnp no)
 		(fields_autoplaced yes)
-		(property "Reference" "C604"
+		(property "Reference" "C601"
 			(at 88.8936 21.59 90)
 			(effects
@@
 			(project "circuit"
 				(path "/420e3d7a-6c9a-4806-b4be-05d56aeb21de/badefe61-f2aa-4ce3-b43f-f44172d96524"
-					(reference "C604")
+					(reference "C601")
 					(unit 1)
 				)
@@
 		(on_board yes)
 		(dnp no)
-		(property "Reference" "#PWR0607"
+		(property "Reference" "#PWR0606"
 			(at 203.2 92.71 0)
 			(effects
@@
 			(project "circuit"
 				(path "/420e3d7a-6c9a-4806-b4be-05d56aeb21de/badefe61-f2aa-4ce3-b43f-f44172d96524"
-					(reference "#PWR0607")
+					(reference "#PWR0606")
 					(unit 1)
 				)
@@
 		(dnp no)
 		(fields_autoplaced yes)
-		(property "Reference" "C606"
+		(property "Reference" "C602"
 			(at 168.9036 21.59 90)
 			(effects
@@
 			(project "circuit"
 				(path "/420e3d7a-6c9a-4806-b4be-05d56aeb21de/badefe61-f2aa-4ce3-b43f-f44172d96524"
-					(reference "C606")
+					(reference "C602")
 					(unit 1)
 				)
@@
 		(dnp no)
 		(fields_autoplaced yes)
-		(property "Reference" "C601"
+		(property "Reference" "C604"
 			(at 60.9536 67.31 90)
 			(effects
@@
 			(project ""
 				(path "/420e3d7a-6c9a-4806-b4be-05d56aeb21de/badefe61-f2aa-4ce3-b43f-f44172d96524"
-					(reference "C601")
+					(reference "C604")
 					(unit 1)
 				)
@@
 		(on_board yes)
 		(dnp no)
-		(property "Reference" "#PWR0602"
+		(property "Reference" "#PWR0608"
 			(at 54.61 181.61 0)
 			(effects
@@
 			(project "circuit"
 				(path "/420e3d7a-6c9a-4806-b4be-05d56aeb21de/badefe61-f2aa-4ce3-b43f-f44172d96524"
-					(reference "#PWR0602")
+					(reference "#PWR0608")
 					(unit 1)
 				)
@@
 		(dnp no)
 		(fields_autoplaced yes)
-		(property "Reference" "U603"
+		(property "Reference" "U602"
 			(at 154.5433 30.48 0)
 			(effects
@@
 			(project "circuit"
 				(path "/420e3d7a-6c9a-4806-b4be-05d56aeb21de/badefe61-f2aa-4ce3-b43f-f44172d96524"
-					(reference "U603")
+					(reference "U602")
 					(unit 1)
 				)
@@
 		(dnp no)
 		(fields_autoplaced yes)
-		(property "Reference" "U604"
+		(property "Reference" "U603"
 			(at 225.6633 30.48 0)
 			(effects
@@
 			(project "circuit"
 				(path "/420e3d7a-6c9a-4806-b4be-05d56aeb21de/badefe61-f2aa-4ce3-b43f-f44172d96524"
-					(reference "U604")
+					(reference "U603")
 					(unit 1)
 				)
@@
 		(on_board yes)
 		(dnp no)
-		(property "Reference" "#PWR0603"
+		(property "Reference" "#PWR0607"
 			(at 96.52 123.19 0)
 			(effects
@@
 			(project "circuit"
 				(path "/420e3d7a-6c9a-4806-b4be-05d56aeb21de/badefe61-f2aa-4ce3-b43f-f44172d96524"
-					(reference "#PWR0603")
-					(unit 1)
-				)
+					(reference "#PWR0607")
+					(unit 1)
+				)
