File: io_routing.kicad_sch (KiCad schematic)
At the start: 7 parts, among them U401 ADG419BN, U402 CD4051B

Commit message: Removed un-needed inhibit from amp out. thereby simplifying the shift registers.
Connections:
- net U901_Q0 is gone; now on net AGND: U402.6 (INH)
Changed lines of the file:
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@@
+	)
+	(junction
+		(at 186.69 95.25)
+		(diameter 0)
+		(color 0 0 0 0)
 	)
 	(junction
@@
 	)
 	(bus_entry
-		(at 147.32 69.85)
-		(size 2.54 2.54)
-		(stroke
-			(width 0)
-			(type default)
-		)
-	)
-	(bus_entry
 		(at 175.26 62.23)
 		(size 2.54 2.54)
@@
 	(wire
 		(pts
-			(xy 149.86 72.39) (xy 186.69 72.39)
-		)
-		(stroke
-			(width 0)
-			(type default)
-		)
-	)
-	(wire
-		(pts
 			(xy 186.69 95.25) (xy 189.23 95.25)
 		)
@@
 		)
 	)
-	(bus
-		(pts
-			(xy 147.32 49.53) (xy 147.32 69.85)
-		)
-		(stroke
-			(width 0)
-			(type default)
-		)
-	)
 	(wire
 		(pts
@@
 		(pts
 			(xy 154.94 167.64) (xy 146.05 167.64)
+		)
+		(stroke
+			(width 0)
+			(type default)
+		)
+	)
+	(wire
+		(pts
+			(xy 186.69 72.39) (xy 186.69 95.25)
 		)
 		(stroke
@@
 	(label "U901_Q[0..4]"
 		(at 147.32 49.53 0)
-		(effects
-			(font
-				(size 1.27 1.27)
-			)
-			(justify left bottom)
-		)
-	)
-	(label "U901_Q0"
-		(at 177.8 72.39 0)
 		(effects
 			(font
@@
 		)
 	)
-	(hierarchical_label "U901_Q[0..4]"
-		(shape output)
-		(at 147.32 52.07 0)
-		(effects
-			(font
-				(size 1.27 1.27)
-			)
-			(justify left)
-		)
-	)

Commit message: Removed LED Shift registers and replaced them with PCA9685 PWM controllers, Also changed LEDs to RGB LEDs.
Parts:
- renumbered C405 to C401, C404 to C402, C401 to C404, C402 to C405, U402 to U401, U401 to U402
Changed lines of the file:
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@@
 		(on_board yes)
 		(dnp no)
-		(property "Reference" "C401"
+		(property "Reference" "C404"
 			(at 125.73 153.6764 90)
 			(effects
@@
 			(project ""
 				(path "/420e3d7a-6c9a-4806-b4be-05d56aeb21de/eb40e95c-c2ba-417c-afee-eaf028752aed"
-					(reference "C401")
+					(reference "C404")
 					(unit 1)
 				)
@@
 		(dnp no)
 		(fields_autoplaced yes)
-		(property "Reference" "U401"
+		(property "Reference" "U402"
 			(at 143.51 113.03 0)
 			(effects
@@
 			(project ""
 				(path "/420e3d7a-6c9a-4806-b4be-05d56aeb21de/eb40e95c-c2ba-417c-afee-eaf028752aed"
-					(reference "U401")
+					(reference "U402")
 					(unit 1)
 				)
@@
 		(dnp no)
 		(fields_autoplaced yes)
-		(property "Reference" "U401"
+		(property "Reference" "U402"
 			(at 151.13 153.6699 0)
 			(effects
@@
 			(project ""
 				(path "/420e3d7a-6c9a-4806-b4be-05d56aeb21de/eb40e95c-c2ba-417c-afee-eaf028752aed"
-					(reference "U401")
+					(reference "U402")
 					(unit 2)
 				)
@@
 		(on_board yes)
 		(dnp no)
-		(property "Reference" "#PWR0403"
+		(property "Reference" "#PWR0401"
 			(at 222.25 57.15 0)
 			(effects
@@
 			(project "circuit"
 				(path "/420e3d7a-6c9a-4806-b4be-05d56aeb21de/eb40e95c-c2ba-417c-afee-eaf028752aed"
-					(reference "#PWR0403")
+					(reference "#PWR0401")
 					(unit 1)
 				)
@@
 		(on_board yes)
 		(dnp no)
-		(property "Reference" "#PWR0401"
+		(property "Reference" "#PWR0403"
 			(at 143.51 187.96 0)
 			(effects
@@
 			(project "circuit"
 				(path "/420e3d7a-6c9a-4806-b4be-05d56aeb21de/eb40e95c-c2ba-417c-afee-eaf028752aed"
-					(reference "#PWR0401")
+					(reference "#PWR0403")
 					(unit 1)
 				)
@@
 		(on_board yes)
 		(dnp no)
-		(property "Reference" "C404"
+		(property "Reference" "C402"
 			(at 191.7636 88.9 90)
 			(effects
@@
 			(project "circuit"
 				(path "/420e3d7a-6c9a-4806-b4be-05d56aeb21de/eb40e95c-c2ba-417c-afee-eaf028752aed"
-					(reference "C404")
+					(reference "C402")
 					(unit 1)
 				)
@@
 		(on_board yes)
 		(dnp no)
-		(property "Reference" "C402"
+		(property "Reference" "C405"
 			(at 148.59 170.1864 90)
 			(effects
@@
 			(project "circuit"
 				(path "/420e3d7a-6c9a-4806-b4be-05d56aeb21de/eb40e95c-c2ba-417c-afee-eaf028752aed"
-					(reference "C402")
+					(reference "C405")
 					(unit 1)
 				)
@@
 		(on_board yes)
 		(dnp no)
-		(property "Reference" "C405"
+		(property "Reference" "C401"
 			(at 210.8136 44.45 90)
 			(effects
@@
 			(project "circuit"
 				(path "/420e3d7a-6c9a-4806-b4be-05d56aeb21de/eb40e95c-c2ba-417c-afee-eaf028752aed"
-					(reference "C405")
+					(reference "C401")
 					(unit 1)
 				)
@@
 		(dnp no)
 		(fields_autoplaced yes)
-		(property "Reference" "U402"
+		(property "Reference" "U401"
 			(at 204.0733 52.07 0)
 			(effects
@@
 			(project "circuit"
 				(path "/420e3d7a-6c9a-4806-b4be-05d56aeb21de/eb40e95c-c2ba-417c-afee-eaf028752aed"
-					(reference "U402")
-					(unit 1)
-				)
+					(reference "U401")
+					(unit 1)
+				)

Commit message: Added Datasheets and specified polyfuse parameters.
Parts:
- U402: value ADG419BN -> ADG419BNZ
Changed lines of the file:
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@@
 			)
 		)
-		(property "Value" "ADG419BN"
+		(property "Value" "ADG419BNZ"
 			(at 143.51 115.57 0)
 			(effects
@@
 			)
 		)
-		(property "Value" "ADG419BN"
+		(property "Value" "ADG419BNZ"
 			(at 151.13 156.2099 0)
 			(effects
